Commit message: fix height fer

File: hpp_control/urdf/fer.urdf (robot description, URDF)
Before this commit: robot fer, 18 links, 17 joints
Links:
- link support_link: geometry collision box size=0.3 0.3 0.01; collision box size=1.703 0.803 0.76
Joints:
- joint support_joint: origin xyz=0.568 -0.1655 .78 rpy=0 0 3.14156 -> xyz=0.568 -0.1655 .77 rpy=0 0 3.14156
